Commit message: got decent example of point to point nav working with lidar and now moving towards exploration mode

File: slam_ws/src/elegoo_description/urdf/elegoo.urdf.xacro (robot description, xacro)
@@ -1,10 +1,40 @@
 <?xml version="1.0"?>
 <robot name="elegoo_minimal" xmlns:xacro="http://www.ros.org/wiki/xacro">
-  <!-- Simple base link (chassis) -->
+  <!--
+    Coordinate convention:
+      +x points forward, +y points left, +z points up.
+      base_link is centered on the chassis footprint.
+    Measure these from the center of the chassis in meters, then update the
+    properties below. Rough values are okay for first bring-up.
+  -->
+  <xacro:property name="chassis_length" value="0.23"/>
+  <xacro:property name="chassis_width"  value="0.13"/>
+  <xacro:property name="chassis_height" value="0.23"/>
+  <xacro:property name="camera_x" value="0.125"/>
+  <xacro:property name="camera_y" value="0.07"/>
+  <xacro:property name="camera_z" value="0.08"/>
+  <xacro:property name="camera_roll"  value="0.0"/>
+  <xacro:property name="camera_pitch" value="0.0"/>
+  <xacro:property name="camera_yaw"   value="0.0"/>
+  <xacro:property name="imu_x" value="-0.11"/>
+  <xacro:property name="imu_y" value="0.00"/>
+  <xacro:property name="imu_z" value="0.14"/>
+  <xacro:property name="imu_roll"  value="0.0"/>
+  <xacro:property name="imu_pitch" value="0.0"/>
+  <xacro:property name="imu_yaw"   value="0.0"/>
+  <xacro:property name="laser_x" value="0.00"/>
+  <xacro:property name="laser_y" value="0.00"/>
+  <xacro:property name="laser_z" value="0.22"/>
+  <xacro:property name="laser_roll"  value="0.0"/>
+  <xacro:property name="laser_pitch" value="0.0"/>
+  <xacro:property name="laser_yaw"   value="0.0"/>
+  <!-- RPLidar is mounted 180 degrees from the robot's +x/front direction. -->
+  <xacro:property name="laser_yaw"   value="3.141592653589793"/>
+  <!-- Chassis -->
   <link name="base_link">
     <visual>
       <origin xyz="0 0 0" rpy="0 0 0"/>
       <geometry>
-        <box size="0.25 0.15 0.05"/>
+        <box size="${chassis_length} ${chassis_width} ${chassis_height}"/>
       </geometry>
       <material name="blue">
@@ -13,5 +43,5 @@
     </visual>
   </link>
-  <!-- LiDAR link: matches your rplidar _frame_id:=laser -->
+  <!-- LiDAR link: matches your rplidar frame_id:=laser -->
   <link name="laser">
     <visual>
@@ -28,7 +58,6 @@
     <parent link="base_link"/>
     <child link="laser"/>
-    <!-- TODO: put the REAL LiDAR position here -->
-    <!-- Example: 10 cm forward, 5 cm above base_link center -->
-    <origin xyz="0.10 0.0 0.05" rpy="0 0 0"/>
+    <origin xyz="${laser_x} ${laser_y} ${laser_z}"
+            rpy="${laser_roll} ${laser_pitch} ${laser_yaw}"/>
   </joint>
   <!-- Realsense camera base frame -->
@@ -47,7 +76,24 @@
     <parent link="base_link"/>
     <child link="camera_link"/>
-    <!-- TODO: real camera position -->
-    <!-- Example: slightly more forward & higher than LiDAR -->
-    <origin xyz="0.12 0.0 0.08" rpy="0 0 0"/>
+    <origin xyz="${camera_x} ${camera_y} ${camera_z}"
+            rpy="${camera_roll} ${camera_pitch} ${camera_yaw}"/>
+  </joint>
+  <!-- IMU frame: matches cmdvel_to_arduino.py imu_frame:=imu_link -->
+  <link name="imu_link">
+    <visual>
+      <origin xyz="0 0 0" rpy="0 0 0"/>
+      <geometry>
+        <box size="0.025 0.025 0.005"/>
+      </geometry>
+      <material name="green">
+        <color rgba="0 0.8 0.2 1"/>
+      </material>
+    </visual>
+  </link>
+  <joint name="imu_joint" type="fixed">
+    <parent link="base_link"/>
+    <child link="imu_link"/>
+    <origin xyz="${imu_x} ${imu_y} ${imu_z}"
+            rpy="${imu_roll} ${imu_pitch} ${imu_yaw}"/>
   </joint>
 </robot>
